Commit message: Update: Added new files and folders to src

File: src/durian_inspection_pkg/urdf/robot.urdf (robot description, URDF)
Before this commit: robot durian_bot, 5 links, 4 joints
Links:
- added link caster_wheel, mass 0.1; collision sphere radius=0.02; visual sphere radius=0.02
- link left_wheel: mass 0.5 -> 1.0; geometry collision sphere radius=0.05; visual cylinder length=0.02 radius=0.05
- link right_wheel: mass 0.5 -> 1.0; geometry collision sphere radius=0.05; visual cylinder length=0.02 radius=0.05
Joints:
- added joint caster_joint: type fixed, parent base_link, child caster_wheel, origin xyz=0.15 0.0 -0.04 rpy=0 0 0
- joint laser_joint: origin xyz=0.12 0.0 0.25 rpy=0 0 0 -> xyz=0.12 0.0 0.26 rpy=0 0 0
- joint left_wheel_joint: origin xyz=-0.1 0.15 0.0 rpy=-1.5708 0 0 -> xyz=0.0 0.18 -0.02 rpy=-1.5708 0 0
- joint right_wheel_joint: origin xyz=-0.1 -0.15 0.0 rpy=-1.5708 0 0 -> xyz=0.0 -0.18 -0.02 rpy=-1.5708 0 0
