Commit message: Update durian inspection ROS2 system

File: src/durian_inspection_pkg/urdf/robot.urdf (robot description, URDF)
Before this commit: robot durian_bot, 6 links, 5 joints
Links:
- removed link caster_wheel
- removed link left_wheel
- removed link right_wheel
- added link base_footprint, mass 0.001
- added link camera_link_optical, mass 0.0001
- link base_link: mass 5.0 -> None
- link camera_link: mass None -> 0.05; geometry collision box size=0.02 0.08 0.03; visual box size=0.02 0.08 0.03
- link laser: geometry collision cylinder length=0.04 radius=0.03; visual cylinder length=0.04 radius=0.03
Joints:
- removed joint caster_joint
- removed joint left_wheel_joint
- removed joint right_wheel_joint
- added joint base_joint: type fixed, parent base_footprint, child base_link, origin xyz=0 0 0.05
- added joint camera_optical_joint: type fixed, parent camera_link, child camera_link_optical, origin xyz=0 0 0 rpy=-1.5708 0 -1.5708
- joint camera_joint: origin xyz=0.18 0.0 0.2 rpy=0 0 0 -> xyz=0.2 0 0.16 rpy=0 0 0
- joint laser_joint: origin xyz=0.12 0.0 0.26 rpy=0 0 0 -> xyz=0.25 0.0 0.8 rpy=0 0 0

Commit message: Update durian inspection pipelines and Flutter app

File: src/durian_inspection_pkg/urdf/robot.urdf (robot description, URDF)
Before this commit: robot durian_bot, 5 links, 4 joints
Links:
- link camera_link: mass 0.05 -> None
Joints:
- joint camera_joint: origin xyz=0.2 0 0.16 rpy=0 0 0 -> xyz=0.25 0 0.8 rpy=0 -0.5236 0
